File: hardware-rj45/can-nano-shield-rj45.kicad_pcb (KiCad board)
At the start: 4 copper layers, 58.5 x 18 mm, 40 parts, among them J1 SSQ-115-03-T-S, J2 SSQ-115-03-T-S, J3 Conn_01x04_Pin, J4 8P8C_LED_Shielded, Q1 AO3401A, T1 B82789C0113N002, U1 MCP2515-xSO, U2 TJA1051T-3, U3 TPSM33625RDNR, Y1 16MHz 9pF

Commit message: minor: minor update before split of rj45
Parts:
- removed JP7: SolderJumper_2_Bridged, Jumper:SolderJumper-2_P1.3mm_Bridged_RoundedPad1.0x1.5mm
Connections:
- J1 pad 05: /CAN_INT_DEFAULT -> /ESTOP
- J1 pad 06: /SYNC -> /CAN_INT_DEFAULT
- J1 pad 08: /ESTOP -> /D5
- J4 pad 4: /CAN_SYNC -> GND
Routing:
- net /CAN_SYNC: track 17.3 -> 0.00 mm
- net /SYNC: track 16.2 -> 0.00 mm, vias 1 -> 0
- net /ESTOP: track 19.2 -> 11.7 mm
- net GND: track 109.3 -> 111.5 mm
- net /CAN_INT_DEFAULT: track 2.71 -> 4.02 mm
