File: hardware-rj45/can-nano-shield-rj45.kicad_sch (KiCad schematic)
At the start: 31 parts, among them J1 SSQ-115-03-T-S, J2 SSQ-115-03-T-S, J3 Conn_01x04_Pin, J4 8P8C_LED_Shielded, Q1 AO3401A, T1 B82789C0113N002, U1 MCP2515-xSO, U2 TJA1051T-3, Y1 16MHz 9pF

Commit message: minor: minor update before split of rj45
Parts:
- removed JP7: SolderJumper_2_Bridged, Jumper:SolderJumper-2_P1.3mm_Bridged_RoundedPad1.0x1.5mm, symbol Jumper:SolderJumper_2_Bridged
Connections:
- net CAN_SYNC is gone; now on net GND: J4.4
- net SYNC is gone; now on net CAN_INT_DEFAULT: A1.6 (D3), J1.06
- net CAN_INT_DEFAULT: no longer A1.5 (D2), J1.05
- net ESTOP: now also A1.5 (D2), J1.05; no longer A1.8 (D5), J1.08
- net RST1: no longer A1.3 (~{RESET}), J1.03
- net RST2 renamed ~{RST2}
- new net D5: A1.8 (D5), J1.08
- new net ~{RST1}: A1.3 (~{RESET}), J1.03
Other:
- note added: "ESTOP"
- note added: "INT"
- note added: "SYNC"
- note added: "Slice:"
