File: hardware/can-nano-shield-rj45.kicad_pcb (KiCad board)
At the start: 4 copper layers, 58.5 x 18 mm, 39 parts, among them J1 SSQ-115-03-T-S, J2 SSQ-115-03-T-S, J3 Conn_01x04_Pin, J4 8P8C_LED_Shielded, Q1 AO3401A, T1 B82789C0113N002, U1 MCP2515-xSO, U2 TJA1051T-3, U3 TPSM33625RDNR, Y1 16MHz 9pF

Commit message: docs: initial commit of docs using slice-infra
Routing:
- net GND: track 111.5 -> 113.0 mm
Changed lines of the file:
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@@
+	)
+	(segment
+		(start 160.48 91.79)
+		(end 160.47 91.79)
+		(width 0.2)
+		(layer "B.Cu")
+		(net 16)
 	)
 	(segment
@@
 	(segment
 		(start 154.189975 90.77)
-		(end 162.26 90.77)
+		(end 159.45 90.77)
 		(width 0.2)
 		(layer "B.Cu")
@@
 	)
 	(segment
+		(start 160.47 91.79)
+		(end 159.45 90.77)
+		(width 0.2)
+		(layer "B.Cu")
+		(net 16)
+	)
+	(segment
 		(start 143.919347 87.045)
 		(end 145.595 87.045)
@@
 		(layer "B.Cu")
 		(net 16)
+	)
+	(segment
+		(start 159.45 90.77)
+		(end 162.26 90.77)
+		(width 0.2)
+		(layer "B.Cu")
+		(net 16)
