File: hardware/can-nano-shield-rj45.kicad_sch (KiCad schematic)
At the start: 30 parts, among them J1 SSQ-115-03-T-S, J2 SSQ-115-03-T-S, J3 Conn_01x04_Pin, J4 8P8C_LED_Shielded, Q1 AO3401A, T1 B82789C0113N002, U1 MCP2515-xSO, U2 TJA1051T-3, Y1 16MHz 9pF

Commit message: docs: initial commit of docs using slice-infra
Connections:
- net RST1 is gone; now on net ~{RST1}: JP4.1 (A)
Changed lines of the file:
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@@
+		)
+	)
+	(label "~{RST1}"
+		(at 123.19 180.34 0)
+		(effects
+			(font
+				(size 1.27 1.27)
+			)
+			(justify left bottom)
 		)
 	)
@@
 			)
 			(justify left bottom)
-		)
-	)
-	(label "RST1"
-		(at 123.19 180.34 0)
-		(effects
-			(font
-				(size 1.27 1.27)
-			)
-			(justify left bottom)
